File: hw/panoptic_platypus/panoptic_platypus.sch (KiCad schematic (older format))
At the start: 3 parts, among them U1 MAX2851, U10 ECP5_5G_25_CABGA381

Commit message: updated power scheme
Connections:
- net LO_Generator 1/REF_CLK_IN: now also U1.50 (CLKOUT2)
- net LO_Generator 2/REF_CLK_IN: now also U1.51 (CLKOUT)
- net Power/VCC_18_0 renamed DRVDD
- no-connect marks 12 -> 8
Changed lines of the file:
@@
 F18 "OEB" I R 8900 3300 50
 F19 "CSB" I R 8900 3700 50
+F20 "DRVDD" I L 8000 2650 50
+F21 "AVDD" I L 8000 2750 50
 $EndSheet
 $Sheet
@@
 F18 "OEB" I R 8900 4850 50
 F19 "CSB" I R 8900 5250 50
+F20 "DRVDD" I L 8000 4200 50
+F21 "AVDD" I L 8000 4300 50
 $EndSheet
 $Sheet
@@
 F18 "OEB" I R 8900 1750 50
 F19 "CSB" I R 8900 2150 50
+F20 "DRVDD" I L 8000 1100 50
+F21 "AVDD" I L 8000 1200 50
 $EndSheet
 $Sheet
@@
 F18 "OEB" I R 8900 6400 50
 F19 "CSB" I R 8900 6800 50
-$EndSheet
-$Sheet
-S 850  950  700  900
-U 5F7981CF
-F0 "Power" 50
-F1 "power.sch" 50
-F2 "Vin" I L 850 1100 50
-F3 "VCC_33" O R 1550 1200 50
-F4 "VCC_50" O R 1550 1050 50
-F5 "VCC_18_0" O R 1550 1350 50
-F6 "VCC_18_1" O R 1550 1500 50
-F7 "VCC_18_2" O R 1550 1650 50
+F20 "DRVDD" I L 8000 5750 50
+F21 "AVDD" I L 8000 5850 50
 $EndSheet
 $Sheet
@@
 	9550 4350 9650 4250
 Wire Bus Line
-	12850 4950 9950 4950
+	12850 5200 9950 5200
 Text Label 12950 1650 0    50   ~ 0
 I_OUT_B0
@@
 Text Label 12950 9750 0    50   ~ 0
 Q_OUT_C15
-Wire Wire Line
-	4100 7050 3950 7050
-Wire Wire Line
-	3950 5550 4000 5550
-Wire Wire Line
-	4200 5550 4200 6900
-Wire Wire Line
-	4200 6900 3950 6900
 Text Label 2400 5950 0    50   ~ 0
 LO_A+
@@
 	2200 7500 2700 7500
 Wire Wire Line
-	2700 5550 2650 5550
-Wire Wire Line
-	2300 5550 2300 6900
-Wire Wire Line
 	2300 6900 2700 6900
 $Comp
@@
 $EndComp
 Wire Bus Line
-	9950 2700 9950 4950
-Wire Bus Line
-	9850 4250 9850 5050
-Wire Bus Line
-	9850 5050 12850 5050
+	9950 2700 9950 5200
+Wire Bus Line
+	9850 4250 9850 5300
+Wire Bus Line
+	9850 5300 12850 5300
 Wire Bus Line
 	8900 1250 9550 1250
@@
 Wire Bus Line
 	8900 5900 9550 5900
-Wire Wire Line
-	4150 4800 4100 4800
 $Comp
 L power:GND #PWR01
@@
 	7250 1350 8000 1350
 Wire Wire Line
-	6700 3300 6950 3300
-Wire Wire Line
-	6950 6300 8000 6300
-Wire Wire Line
-	6950 3300 6950 6300
-Wire Wire Line
-	8000 6200 7000 6200
-Wire Wire Line
-	7000 6200 7000 3200
-Wire Wire Line
-	7000 3200 6700 3200
-Wire Wire Line
-	6700 3100 7050 3100
-Wire Wire Line
-	7050 3100 7050 6100
-Wire Wire Line
-	7050 6100 8000 6100
-Wire Wire Line
-	8000 6000 7100 6000
-Wire Wire Line
-	7100 6000 7100 3000
-Wire Wire Line
-	7100 3000 6700 3000
-Wire Wire Line
-	6700 2850 7200 2850
-Wire Wire Line
-	7200 2850 7200 4750
-Wire Wire Line
-	7200 4750 8000 4750
-Wire Wire Line
-	8000 4650 7250 4650
-Wire Wire Line
-	7250 4650 7250 2750
-Wire Wire Line
-	7250 2750 6700 2750
-Wire Wire Line
-	6700 2650 7300 2650
-Wire Wire Line
-	7300 2650 7300 4550
-Wire Wire Line
-	7300 4550 8000 4550
-Wire Wire Line
-	8000 4450 7350 4450
-Wire Wire Line
-	7350 4450 7350 2550
-Wire Wire Line
-	7350 2550 6700 2550
-Wire Wire Line
-	6700 2400 7450 2400
-Wire Wire Line
-	7450 2400 7450 3200
-Wire Wire Line
-	7450 3200 8000 3200
-Wire Wire Line
-	8000 3100 7500 3100
-Wire Wire Line
-	7500 3100 7500 2300
-Wire Wire Line
-	7500 2300 6700 2300
-Wire Wire Line
-	6700 2200 7550 2200
-Wire Wire Line
-	7550 2200 7550 3000
-Wire Wire Line
-	7550 3000 8000 3000
-Wire Wire Line
-	8000 2900 7600 2900
-Wire Wire Line
-	7600 2900 7600 2100
-Wire Wire Line
-	7600 2100 6700 2100
-NoConn ~ 6700 3450
-NoConn ~ 6700 3550
-NoConn ~ 6700 3650
-NoConn ~ 6700 3750
+	6700 3300 7000 3300
+Wire Wire Line
+	7000 6300 8000 6300
+Wire Wire Line
+	7000 3300 7000 6300
+Wire Wire Line
+	8000 6200 7050 6200
+Wire Wire Line
+	7050 6200 7050 3200
+Wire Wire Line
+	7050 3200 6700 3200
+Wire Wire Line
+	6700 3100 7100 3100
+Wire Wire Line
+	7100 3100 7100 6100
+Wire Wire Line
+	7100 6100 8000 6100
+Wire Wire Line
+	8000 6000 7150 6000
+Wire Wire Line
+	7150 6000 7150 3000
+Wire Wire Line
+	7150 3000 6700 3000
+Wire Wire Line
+	6700 2850 7250 2850
+Wire Wire Line
+	7250 2850 7250 4750
+Wire Wire Line
+	7250 4750 8000 4750
+Wire Wire Line
+	8000 4650 7300 4650
+Wire Wire Line
+	7300 4650 7300 2750
+Wire Wire Line
+	7300 2750 6700 2750
+Wire Wire Line
+	6700 2650 7350 2650
+Wire Wire Line
+	7350 2650 7350 4550
+Wire Wire Line
+	7350 4550 8000 4550
+Wire Wire Line
+	6700 2400 7500 2400
+Wire Wire Line
+	7500 3200 8000 3200
+Wire Wire Line
+	8000 3100 7550 3100
+Wire Wire Line
+	7550 3100 7550 2300
+Wire Wire Line
+	7550 2300 6700 2300
+Wire Wire Line
+	6700 2200 7600 2200
+Wire Wire Line
+	7600 2200 7600 3000
+Wire Wire Line
+	7600 3000 8000 3000
+Wire Wire Line
+	8000 2900 7650 2900
+Wire Wire Line
+	7650 2900 7650 2100
+Wire Wire Line
+	7650 2100 6700 2100
 NoConn ~ 6700 3900
 NoConn ~ 6700 4000
@@
 Wire Wire Line
 	15350 950  15250 950
-Wire Wire Line
-	2650 950  2650 1350
-Wire Wire Line
-	2650 1350 1550 1350
 Connection ~ 11850 950
-Wire Wire Line
-	11850 950  2650 950
 Connection ~ 11950 950
 Wire Wire Line
@@
 Connection ~ 15150 950
 Wire Wire Line
-	15150 950  12150 950
+	15150 950  12350 950
 Connection ~ 15250 950
 Wire Wire Line
 	15250 950  15150 950
 Wire Wire Line
-	12150 950  12150 5950
-Wire Wire Line
-	12150 5950 12350 5950
-Connection ~ 12150 950
-Wire Wire Line
-	12150 950  11950 950
+	12350 950  12350 5950
+Connection ~ 12350 950
+Wire Wire Line
+	12350 950  11950 950
 Connection ~ 12350 5950
 Wire Wire Line
@@
 Wire Bus Line
 	1850 2850 1800 8100
-Wire Wire Line
-	2650 5550 2650 5300
-Wire Wire Line
-	2650 5300 3050 5300
-Connection ~ 2650 5550
-Wire Wire Line
-	2650 5550 2300 5550
-Wire Wire Line
-	4000 5550 4000 5300
-Wire Wire Line
-	4000 5300 3550 5300
-Connection ~ 4000 5550
-Wire Wire Line
-	4000 5550 4200 5550
+$Sheet
+S 850  900  700  900
+U 5F7981CF
+F0 "Power" 50
+F1 "power.sch" 50
+F2 "Vin" I L 850 1050 50
+F3 "VCC_50" O R 1550 1550 50
+F4 "VCC_18_0" O R 1550 950 50
+F5 "VCC_18_1" O R 1550 1050 50
+F6 "VCC_18_2" O R 1550 1150 50
+F7 "VCC_33_0" O R 1550 1450 50
+F8 "VCC_33_1" O R 1550 1250 50
+F9 "VCC_33_2" O R 1550 1350 50
+$EndSheet
+Wire Wire Line
+	1550 950  11850 950
+Wire Wire Line
+	8000 2650 7750 2650
+Wire Wire Line
+	8000 2750 7750 2750
+Text Label 7750 2650 0    50   ~ 0
+DRVDD
+Wire Wire Line
+	8000 1100 7750 1100
+Wire Wire Line
+	8000 1200 7750 1200
+Text Label 7750 1100 0    50   ~ 0
+DRVDD
+Wire Wire Line
+	8000 4200 7750 4200
+Wire Wire Line
+	8000 4300 7750 4300
+Text Label 7750 4200 0    50   ~ 0
+DRVDD
+Text Label 7750 4300 0    50   ~ 0
+AVDD1
+Wire Wire Line
+	8000 5750 7750 5750
+Wire Wire Line
+	8000 5850 7750 5850
+Text Label 7750 5750 0    50   ~ 0
+DRVDD
+Text Label 7750 5850 0    50   ~ 0
+AVDD1
+Text Label 1800 950  0    50   ~ 0
+DRVDD
+Text Label 7750 2750 0    50   ~ 0
+AVDD0
+Text Label 7750 1200 0    50   ~ 0
+AVDD0
+Wire Wire Line
+	3950 5550 4450 5550
+Wire Wire Line
+	2300 5550 2700 5550
+Wire Wire Line
+	7500 2400 7500 3200
+Wire Wire Line
+	7400 2550 6700 2550
+Wire Wire Line
+	8000 4450 7400 4450
+Wire Wire Line
+	7400 4450 7400 2550
+Wire Wire Line
+	6700 3450 6900 3450
+Wire Wire Line
+	6900 3450 6900 4350
+Wire Wire Line
+	6700 3550 6850 3550
+Wire Wire Line
+	6850 3550 6850 4350
+Wire Wire Line
+	6700 3650 6800 3650
+Wire Wire Line
+	6800 3650 6800 4350
+Wire Wire Line
+	6700 3750 6750 3750
+Wire Wire Line
+	6750 3750 6750 4350
+Wire Wire Line
+	3950 5700 4000 5700
+Wire Wire Line
+	4000 5700 4000 4800
+Wire Wire Line
+	3950 7050 4150 7050
+Wire Wire Line
+	4150 7050 4150 4800
+Text Label 4450 5550 2    50   ~ 0
+DRVDD
+Wire Wire Line
+	3950 6900 4450 6900
+Text Label 4450 6900 2    50   ~ 0
+DRVDD
 Wire Bus Line
 	8900 2700 9950 2700
@@
 	10050 1150 10050 4650
 Wire Bus Line
-	12850 5050 12850 9650
-Wire Bus Line
-	12850 1550 12850 4950
+	12850 5300 12850 9650
+Wire Bus Line
+	12850 1550 12850 5200
 Wire Bus Line
 	10050 5800 10050 9650
