File: hw/panoptic_platypus/power.sch (KiCad schematic (older format))
At the start: 1 part, among them U10 ECP5_5G_25_CABGA381

Commit message: added power supply, connected up some bits
Parts:
- added C? (x24): C_Small, symbol Device:C_Small
- added L? (x4): L_Small, symbol Device:L_Small
- added R? (x10): R_Small, symbol Device:R_Small
- added U? (x2): TPS56339, Package_TO_SOT_SMD:SOT-23-6, symbol dknueppe_symbols:TPS56339
- added U? (x2): TLV62569DDC, Package_TO_SOT_SMD:SOT-23-6, symbol Regulator_Switching:TLV62569DDC
- added U? (x6): MCP1826S, symbol Regulator_Linear:MCP1826S
Connections:
- net GND: now also C?.2, C?.2, C?.2, C?.2, C?.2, C?.2, C?.2, C?.2, C?.2, C?.2, C?.2, C?.2, C?.2, C?.2, C?.2, C?.2, C?.2, C?.2, R?.1, R?.1, R?.2, R?.2, U?.2 (GND), U?.2 (GND), U?.2 (GND), U?.2 (GND), U?.2 (GND), U?.2 (GND), U?.2 (GND), U?.2 (GND)
- net VCC renamed 1.2V
- net 1.2V: now also C?.1, C?.1, L?.2, R?.1; no longer U10.F15 (VCCAUX), U10.F6 (VCCAUX), U10.P15 (VCCAUX), U10.P6 (VCCAUX), U10.V10 (VCCAUXA0), U10.V11 (VCCAUXA0)
- new net: C?.2, U?.1 (GND) (x2)
- new net: C?.2, U?.2 (SW) (x2)
- new net: R?.1, R?.2, U?.4 (FB) (x2)
- new net: R?.2, U?.6 (BOOT) (x2)
- new net: L?.1, U?.3 (SW) (x2)
- new net: C?.2, R?.1, R?.2, U?.6 (FB) (x2)
- new net: C?.1, L?.1, R?.1 (x2)
- new net 2.5V: C?.1, C?.1, C?.1, L?.2, R?.2, U10.F15 (VCCAUX), U10.F6 (VCCAUX), U10.P15 (VCCAUX), U10.P6 (VCCAUX), U10.V10 (VCCAUXA0), U10.V11 (VCCAUXA0), U?.1 (VI), U?.1 (VI)
- new net 5.5V: C?.1, C?.1, C?.1, C?.1, C?.1, C?.1, C?.1, L?.2, R?.2, U?.1 (VI), U?.1 (VI), U?.1 (VI), U?.1 (VI), U?.4 (VIN), U?.4 (VIN)
- new net VCC_18_0: C?.1, C?.1, L?.2, R?.1
- new net VCC_18_1: C?.1, U?.3 (VO)
- new net VCC_18_2: C?.1, U?.3 (VO)
- new net VCC_33_0: C?.1, U?.3 (VO)
- new net VCC_33_1: C?.1, U?.3 (VO)
- new net VCC_33_2: C?.1, U?.3 (VO)
- new net VCC_50: C?.1, U?.3 (VO)
- new net Vin: C?.1, C?.1, U?.3 (VIN), U?.3 (VIN)
Other:
- note added: "2.5 V"
- note added: "5.5 V"
- moved on the sheet: U10A
